File: STM32MP1_TestBoard_RevC/GPIO.sch (KiCad schematic (older format))
At the start: 24 parts, among them J1 Conn_01x27, J2 Conn_01x27, J3 Conn_01x27, J4 Conn_01x27, J5 Conn_02x03_Odd_Even, J7 Conn_01x08, U1 STM32MP157xAB, X1 NX2016SA-24M, Y1 NX2012SA32768K1

Commit message: HW changes
- Changed buck converter(TPS42402) to LDO (AZ1117)
Parts:
- added D5, D6, D7: LED, LED_SMD:LED_0805_2012Metric_Pad1.15x1.40mm_HandSolder, symbol Device:LED
- added J11: Conn_01x06, Connector_PinHeader_2.54mm:PinHeader_1x06_P2.54mm_Vertical, symbol Connector_Generic:Conn_01x06
- added R16, R17, R27: 1K, Resistor_SMD:R_0402_1005Metric_Pad0.72x0.64mm_HandSolder, symbol Device:R
- added TP6, TP7, TP8, TP9: TestPoint, TestPoint:TestPoint_Pad_D1.0mm, symbol Connector:TestPoint
Connections:
- net 3.3V_VDD: now also D5.2 (A), D6.2 (A), D7.2 (A), J11.3 (Pin_3)
- net GNDS: now also J11.1 (Pin_1)
- net PA14: now also R16.1
- net PB2: now also J11.4 (Pin_4), TP9.1
- net PG11: now also J11.5 (Pin_5), TP8.1
- net PG6: now also R17.1
- net PD11 renamed HEARTBEAT_LED
- net HEARTBEAT_LED: now also R27.1
- new net: D5.1 (K), R16.2
- new net: D6.1 (K), R17.2
- new net: J11.2 (Pin_2), TP7.1
- new net: J11.6 (Pin_6), TP6.1
- new net: D7.1 (K), R27.2
Other:
- note added: "Supplied by VDD3V3_USBFS"
- moved on the sheet: C37, D1, NT3, R20, R21, R22, R9, X1
