File: STM32MP1_TestBoard_RevC/Power_MPU.sch (KiCad schematic (older format))
At the start: 33 parts, among them J12 Conn_01x02, U1 STM32MP157xAB

Commit message: HW changes
- Changed buck converter(TPS42402) to LDO (AZ1117)
Parts:
- L3: footprint Inductor_SMD:L_0201_0603Metric_Pad0.64x0.40mm_HandSolder -> Inductor_SMD:L_0603_1608Metric_Pad1.05x0.95mm_HandSolder
Changed lines of the file:
@@
 F 0 "L3" V 10650 2875 50  0000 C CNN
 F 1 "LQM18FN4R7M00D " V 10500 2875 50  0000 C CNN
-F 2 "Inductor_SMD:L_0201_0603Metric_Pad0.64x0.40mm_HandSolder" H 10575 2875 50  0001 C CNN
+F 2 "Inductor_SMD:L_0603_1608Metric_Pad1.05x0.95mm_HandSolder" H 10575 2875 50  0001 C CNN
 F 3 "https://www.mouser.co.uk/datasheet/2/281/JELF243B-0012-1633801.pdf" H 10575 2875 50  0001 C CNN
 F 4 "~" H 10575 2875 50  0001 C CNN "Mfr"
